File: Hardware/interface/interface.kicad_sch (KiCad schematic)
At the start: 21 parts, among them J1 TFmini1, J2 TFmini2, J3 TFmini3, U3 TS5A3357, U4 TXB0102DCT, U5 TS5A3357, U6 ARDUINO_MICRO_SHIELD

Commit message: Almost finish PCB routing
Parts:
- removed U3, U5: TS5A3357, Package_SO:VSSOP-8_3.0x3.0mm_P0.65mm, symbol analogSwitch:TS5A3357
- added unit 1 of U1
- added unit 1 of U2
- U1, U2: value ~ -> TS5A3357
- renumbered C5 to C1, C1 to C11, C2 to C12, C8 to C2, C11 to C3, C6 to C4, C9 to C5, C12 to C6, C3 to C7, C4 to C8, C7 to C9, U4 to U3, U6 to U4
Connections:
- net CMD_1: now also U4.A4, U1.6 (IN1), U2.6 (IN1); no longer U4.A0
- net CMD_2: now also U4.A5, U1.5 (IN2), U2.5 (IN2); no longer U4.A1
- net RX_TF1: now also U1.1 (NO0)
- net RX_TF2: now also U1.2 (NO1)
- net RX_TF3: now also U1.3 (NO2)
- net TX_TF1: now also U2.1 (NO0)
- net TX_TF2: now also U2.2 (NO1)
- net TX_TF3: now also U2.3 (NO2)
- net at U3.5 (A1): now also U1.7 (COM)
- net at U3.4 (A2): now also U2.7 (COM)

Commit message: Change sensor connectors to be more strong, efficient
Parts:
- J1, J2, J3: footprint Connector_PinHeader_2.54mm:PinHeader_1x04_P2.54mm_Vertical -> Connector_Wire:SolderWire-0.1sqmm_1x04_P3.6mm_D0.4mm_OD1mm_Relief
Changed lines of the file:
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@@
 	(label "TX_TF2"
 		(at 35.56 99.06 0)
-		(fields_autoplaced yes)
 		(effects
 			(font
@@
 	(label "RX_TF3"
 		(at 99.06 86.36 180)
-		(fields_autoplaced yes)
 		(effects
 			(font
@@
 	(label "CMD_2"
 		(at 116.84 95.25 270)
-		(fields_autoplaced yes)
 		(effects
 			(font
@@
 	(label "TX_TF3"
 		(at 35.56 123.19 0)
-		(fields_autoplaced yes)
 		(effects
 			(font
@@
 	(label "CMD_2"
 		(at 116.84 127 270)
-		(fields_autoplaced yes)
 		(effects
 			(font
@@
 	(label "TX_TF2"
 		(at 99.06 114.3 180)
-		(fields_autoplaced yes)
 		(effects
 			(font
@@
 	(label "CMD_1"
 		(at 204.47 106.68 180)
-		(fields_autoplaced yes)
 		(effects
 			(font
@@
 	(label "TX_TF1"
 		(at 99.06 110.49 180)
-		(fields_autoplaced yes)
 		(effects
 			(font
@@
 	(label "CMD_1"
 		(at 111.76 95.25 270)
-		(fields_autoplaced yes)
 		(effects
 			(font
@@
 	(label "RX_TF3"
 		(at 35.56 120.65 0)
-		(fields_autoplaced yes)
 		(effects
 			(font
@@
 	(label "RX_TF2"
 		(at 99.06 82.55 180)
-		(fields_autoplaced yes)
 		(effects
 			(font
@@
 	(label "TX"
 		(at 166.37 100.33 0)
-		(fields_autoplaced yes)
 		(effects
 			(font
@@
 	(label "RX_TF1"
 		(at 35.56 73.66 0)
-		(fields_autoplaced yes)
 		(effects
 			(font
@@
 	(label "RX"
 		(at 251.46 124.46 0)
-		(fields_autoplaced yes)
 		(effects
 			(font
@@
 	(label "RX"
 		(at 166.37 95.25 0)
-		(fields_autoplaced yes)
 		(effects
 			(font
@@
 	(label "TX"
 		(at 251.46 121.92 0)
-		(fields_autoplaced yes)
 		(effects
 			(font
@@
 	(label "TX_TF3"
 		(at 99.06 118.11 180)
-		(fields_autoplaced yes)
 		(effects
 			(font
@@
 	(label "RX_TF1"
 		(at 99.06 78.74 180)
-		(fields_autoplaced yes)
 		(effects
 			(font
@@
 	(label "CMD_2"
 		(at 204.47 109.22 180)
-		(fields_autoplaced yes)
 		(effects
 			(font
@@
 	(label "CMD_1"
 		(at 111.76 127 270)
-		(fields_autoplaced yes)
 		(effects
 			(font
@@
 	(label "RX_TF2"
 		(at 35.56 96.52 0)
-		(fields_autoplaced yes)
 		(effects
 			(font
@@
 	(label "TX_TF1"
 		(at 35.56 76.2 0)
-		(fields_autoplaced yes)
 		(effects
 			(font
@@
 			)
 		)
-		(property "Footprint" "Connector_PinHeader_2.54mm:PinHeader_1x04_P2.54mm_Vertical"
+		(property "Footprint" "Connector_Wire:SolderWire-0.1sqmm_1x04_P3.6mm_D0.4mm_OD1mm_Relief"
 			(at 25.4 93.98 0)
 			(effects
@@
 			)
 		)
-		(property "Footprint" "Connector_PinHeader_2.54mm:PinHeader_1x04_P2.54mm_Vertical"
+		(property "Footprint" "Connector_Wire:SolderWire-0.1sqmm_1x04_P3.6mm_D0.4mm_OD1mm_Relief"
 			(at 25.4 118.11 0)
 			(effects
@@
 			)
 		)
-		(property "Footprint" "Connector_PinHeader_2.54mm:PinHeader_1x04_P2.54mm_Vertical"
+		(property "Footprint" "Connector_Wire:SolderWire-0.1sqmm_1x04_P3.6mm_D0.4mm_OD1mm_Relief"
 			(at 25.4 71.12 0)
 			(effects
